File: arduinopic/arduinopic.kicad_pcb (KiCad board)
At the start: 2 copper layers, 78.7 x 48.3 mm, 19 parts, among them Q1 BC847, U1 PIC16F628-xxIP, U2 PIC16F610-IP

Commit message: PIC12F629, PIC12F675 support added
Parts:
- added D1: LED, LED_SMD:LED_1206_3216Metric_Pad1.42x1.75mm_HandSolder, B.Cu at (146.1, 96.5)
- added R6: 1k, Resistor_SMD:R_1206_3216Metric_Pad1.42x1.75mm_HandSolder, B.Cu at (146.1, 101.6)
- added R7: 47R, Resistor_SMD:R_1206_3216Metric_Pad1.42x1.75mm_HandSolder, B.Cu at (129.5, 86.6)
- C2: value 1000uF -> 100nF; footprint Capacitor_THT:CP_Radial_D10.0mm_P5.00mm -> Capacitor_SMD:C_1206_3216Metric_Pad1.42x1.75mm_HandSolder; moved to B.Cu
- moved C2 35.1 mm to (81.3, 110.5), turned to 90 degrees
Connections:
- A1 pad 24: (no net) -> LED
- A1 pad 5: (no net) -> Net-(A1-Pad5)
- C1 pad 1: /VCC -> /VDD1
- C2 pad 1: /VCC -> /VDD2
- S1 pad 2A: /VCC -> Net-(A1-Pad27)
- S1 pad 3A: Net-(A1-Pad27) -> /VDD1
- S1 pad 3B: /5V-Ext -> /VDD
- S1 pad 4A: (no net) -> /VDD2
- S1 pad 4B: (no net) -> /VDD
- U1 pad 14: /VCC -> /VDD1
- U2 pad 1: /VCC -> /VDD2
Routing:
- net /VCC: track 101.3 -> 0.00 mm, vias 2 -> 0
- net /VDD1: track 0.00 -> 91.4 mm, vias 0 -> 2
- net /VDD: track 0.00 -> 67.3 mm
- net /VDD2: track 0.00 -> 41.3 mm
- net Net-(R3-Pad2): track 32.1 -> 16.6 mm
- net Net-(Q1-Pad1): track 58.5 -> 49.5 mm
- net GND: track 223.8 -> 232.5 mm
- net Net-(A1-Pad5): track 0.00 -> 5.52 mm
- net Net-(D1-Pad1): track 0.00 -> 5.08 mm
- net /5V-Ext: track 74.2 -> 69.4 mm
- net /DATA: track 110.4 -> 106.2 mm
- net LED: track 0.00 -> 3.59 mm
- net /Vpp: track 54.1 -> 55.6 mm
- net Net-(A1-Pad27): track 83.4 -> 82.4 mm
Other:
- board text added: "12F"
- board text added: "16F"
- board text removed: "5V"
